File: impednace-analyzer-pcb/hardware/impedance-analyzer/impedance-analyzer.kicad_pcb (KiCad board)
At the start: 2 copper layers, 61.9 x 56.5 mm, 11 parts, among them J1 AD9833, J2 ADS1256_SPI, J3 ADS1256_AIN, J4 UNO_POWER, J5 UNO_ANALOG, J6 UNO_DIGITAL_LOW, J7 UNO_DIGITAL_HIGH, J8 PIEZO

Commit message: pcb stuff
Parts:
- moved J1 99.8 mm to (136.3, 89.8)
Changed lines of the file:
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@@
 	(footprint "Connector_PinSocket_2.54mm:PinSocket_1x07_P2.54mm_Vertical"
 		(layer "F.Cu")
-		(at 231.59 60.21)
+		(at 136.3 89.81)
 		(descr "Through hole straight socket strip, 1x07, 2.54mm pitch, single row (from Kicad 4.0.7), script generated")
 		(tags "Through hole socket strip THT 1x07 2.54mm single row")
