File: impednace-analyzer-pcb/hardware/impedance-analyzer/impedance-analyzer.kicad_sch (KiCad schematic)
At the start: 8 parts, among them U1 AD9833BRMZ, Y1 ABM3-25.000MHZ-J2Y-T

Commit message: did schematic work
Parts:
- removed C1: 100nF, symbol Device:C
- removed C2: 10uF, symbol Device:C
- removed C3, C4: 10nF, symbol Device:C
- removed C5, C6: 22pF, symbol Device:C
- removed U1: AD9833BRMZ, impedance-analyzer:SOP50P490X110-10N, symbol ImpedanceAnalyzer:AD9833BRMZ
- removed Y1: ABM3-25.000MHZ-J2Y-T, ABM3-25.000MHZ-J2Y-T:XTAL_ABM3-25.000MHZ-J2Y-T, symbol ImpedanceAnalyzer:ABM3-25.000MHZ-J2Y-T
- added J1: AD9833, symbol Connector_Generic:Conn_01x07
- added J2: ADS1256_SPI, symbol Connector_Generic:Conn_01x08
- added J3: ADS1256_AIN, symbol Connector_Generic:Conn_02x08_Odd_Even
- added J4: UNO_POWER, symbol Connector_Generic:Conn_01x08
- added J5: UNO_ANALOG, symbol Connector_Generic:Conn_01x06
- added J6: UNO_DIGITAL_LOW, symbol Connector_Generic:Conn_01x08
- added J7: UNO_DIGITAL_HIGH, symbol Connector_Generic:Conn_01x10
- added J8: PIEZO, symbol Connector_Generic:Conn_01x02
- added RV1: R_Potentiometer, symbol Device:R_Potentiometer
Connections:
- net +5V: now also J1.1 (Pin_1), J2.1 (Pin_1), J2.8 (Pin_8), J4.5 (Pin_5)
- net GND: now also J1.2 (Pin_2), J1.6 (Pin_6), J2.2 (Pin_2), J3.15 (Pin_15), J3.16 (Pin_16), J3.2 (Pin_2), J3.4 (Pin_4), J4.6 (Pin_6), J4.7 (Pin_7), J7.7 (Pin_7), J8.2 (Pin_2)
- new net AD9833_OUT: J1.7 (Pin_7), J3.1 (Pin_1), RV1.1
- new net ADC_CS: J2.7 (Pin_7), J7.3 (Pin_3)
- new net DRDY: J2.6 (Pin_6), J7.2 (Pin_2)
- new net FSYNC: J1.5 (Pin_5), J7.1 (Pin_1)
- new net MISO: J2.5 (Pin_5), J7.5 (Pin_5)
- new net SCLK: J1.4 (Pin_4), J2.3 (Pin_3), J7.6 (Pin_6)
- new net SDATA: J1.3 (Pin_3), J2.4 (Pin_4), J7.4 (Pin_4)
- new net VMID_NODE: J3.3 (Pin_3), J8.1 (Pin_1), RV1.2, RV1.3
- no-connect marks 0 -> 32
Other:
- note added: "ADC"
- note added: "Arduino_UNO"
- note added: "Voltage Divider"

Commit message: started pcb layout and design
Changed lines of the file:
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@@
+	)
+	(junction
+		(at 207.01 46.99)
+		(diameter 0)
+		(color 0 0 0 0)
 	)
 	(junction
@@
 	)
 	(junction
+		(at 59.69 33.02)
+		(diameter 0)
+		(color 0 0 0 0)
+	)
+	(junction
 		(at 53.34 160.02)
 		(diameter 0)
@@
 	(wire
 		(pts
-			(xy 53.34 163.83) (xy 53.34 170.18)
+			(xy 59.69 33.02) (xy 66.04 33.02)
 		)
 		(stroke
@@
 	(wire
 		(pts
-			(xy 59.69 154.94) (xy 59.69 160.02)
+			(xy 53.34 163.83) (xy 53.34 170.18)
 		)
 		(stroke
@@
 	(wire
 		(pts
-			(xy 57.15 154.94) (xy 59.69 154.94)
+			(xy 59.69 154.94) (xy 59.69 160.02)
 		)
 		(stroke
@@
 	(wire
 		(pts
-			(xy 143.51 29.21) (xy 151.13 29.21)
+			(xy 57.15 154.94) (xy 59.69 154.94)
 		)
 		(stroke
@@
 	(wire
 		(pts
-			(xy 144.78 46.99) (xy 151.13 46.99)
+			(xy 143.51 29.21) (xy 151.13 29.21)
 		)
 		(stroke
@@
 	(wire
 		(pts
-			(xy 62.23 48.26) (xy 66.04 48.26)
+			(xy 144.78 46.99) (xy 151.13 46.99)
 		)
 		(stroke
@@
 	(wire
 		(pts
-			(xy 53.34 163.83) (xy 62.23 163.83)
+			(xy 62.23 48.26) (xy 66.04 48.26)
 		)
 		(stroke
@@
 	(wire
 		(pts
-			(xy 53.34 142.24) (xy 60.96 142.24)
+			(xy 53.34 163.83) (xy 62.23 163.83)
 		)
 		(stroke
@@
 	(wire
 		(pts
-			(xy 53.34 158.75) (xy 53.34 160.02)
+			(xy 53.34 142.24) (xy 60.96 142.24)
 		)
 		(stroke
@@
 	(wire
 		(pts
-			(xy 53.34 172.72) (xy 53.34 176.53)
+			(xy 53.34 158.75) (xy 53.34 160.02)
 		)
 		(stroke
@@
 	(wire
 		(pts
-			(xy 62.23 38.1) (xy 66.04 38.1)
+			(xy 53.34 172.72) (xy 53.34 176.53)
 		)
 		(stroke
@@
 	(wire
 		(pts
-			(xy 57.15 33.02) (xy 66.04 33.02)
+			(xy 62.23 38.1) (xy 66.04 38.1)
+		)
+		(stroke
+			(width 0)
+			(type default)
+		)
+	)
+	(wire
+		(pts
+			(xy 57.15 33.02) (xy 59.69 33.02)
 		)
 		(stroke
@@
 					(unit 1)
 				)
+			)
+		)
+	)
+	(symbol
+		(lib_id "power:PWR_FLAG")
+		(at 207.01 46.99 180)
+		(unit 1)
+		(body_style 1)
+		(exclude_from_sim no)
+		(in_bom yes)
+		(on_board yes)
+		(in_pos_files yes)
+		(dnp no)
+		(fields_autoplaced yes)
+		(property "Reference" "#FLG02"
+			(at 207.01 48.895 0)
+			(hide yes)
+			(show_name no)
+			(do_not_autoplace no)
+			(effects
+				(font
+					(size 1.27 1.27)
+				)
+			)
+		)
+		(property "Value" "PWR_FLAG"
+			(at 207.01 52.07 0)
+			(show_name no)
+			(do_not_autoplace no)
+			(effects
+				(font
+					(size 1.27 1.27)
+				)
+			)
+		)
+		(property "Footprint" ""
+			(at 207.01 46.99 0)
+			(hide yes)
+			(show_name no)
+			(do_not_autoplace no)
+			(effects
+				(font
+					(size 1.27 1.27)
+				)
+			)
+		)
+		(property "Datasheet" ""
+			(at 207.01 46.99 0)
+			(hide yes)
+			(show_name no)
+			(do_not_autoplace no)
+			(effects
+				(font
+					(size 1.27 1.27)
+				)
+			)
+		)
+		(property "Description" "Special symbol for telling ERC where power comes from"
+			(at 207.01 46.99 0)
+			(hide yes)
+			(show_name no)
+			(do_not_autoplace no)
+			(effects
+				(font
+					(size 1.27 1.27)
+				)
+			)
+		)
+		(pin "1"
+		)
+		(instances
+			(project "impedance-analyzer"
+				(path "/259d1f59-b563-4094-a7dc-8c16a7d2f7ef"
+					(reference "#FLG02")
+					(unit 1)
+				)
+			)
+		)
+	)
+	(symbol
+		(lib_id "power:PWR_FLAG")
+		(at 59.69 33.02 0)
+		(unit 1)
+		(body_style 1)
+		(exclude_from_sim no)
+		(in_bom yes)
+		(on_board yes)
+		(in_pos_files yes)
+		(dnp no)
+		(fields_autoplaced yes)
+		(property "Reference" "#FLG01"
+			(at 59.69 31.115 0)
+			(hide yes)
+			(show_name no)
+			(do_not_autoplace no)
+			(effects
+				(font
+					(size 1.27 1.27)
+				)
+			)
+		)
+		(property "Value" "PWR_FLAG"
+			(at 59.69 27.94 0)
+			(show_name no)
+			(do_not_autoplace no)
+			(effects
+				(font
+					(size 1.27 1.27)
+				)
+			)
+		)
+		(property "Footprint" ""
+			(at 59.69 33.02 0)
+			(hide yes)
+			(show_name no)
+			(do_not_autoplace no)
+			(effects
+				(font
+					(size 1.27 1.27)
+				)
+			)
+		)
+		(property "Datasheet" ""
+			(at 59.69 33.02 0)
+			(hide yes)
+			(show_name no)
+			(do_not_autoplace no)
+			(effects
+				(font
+					(size 1.27 1.27)
+				)
+			)
+		)
+		(property "Description" "Special symbol for telling ERC where power comes from"
+			(at 59.69 33.02 0)
+			(hide yes)
+			(show_name no)
+			(do_not_autoplace no)
+			(effects
+				(font
+					(size 1.27 1.27)
+				)
+			)
+		)
+		(pin "1"
+		)
+		(instances
+			(project "impedance-analyzer"
+				(path "/259d1f59-b563-4094-a7dc-8c16a7d2f7ef"
+					(reference "#FLG01")
+					(unit 1)
+				)

Commit message: pcb stuff
Parts:
- added C1: 100nF, Capacitor_SMD:C_0805_2012Metric_Pad1.18x1.45mm_HandSolder, symbol Device:C
- added C2: 10uF, Capacitor_SMD:C_0805_2012Metric_Pad1.18x1.45mm_HandSolder, symbol Device:C
- J1: footprint (none) -> Connector_PinSocket_2.54mm:PinSocket_1x07_P2.54mm_Vertical
- J2: footprint (none) -> Connector_PinSocket_2.54mm:PinSocket_1x08_P2.54mm_Vertical
- J3: footprint (none) -> Connector_PinSocket_2.54mm:PinSocket_2x08_P2.54mm_Vertical
- J4, J6: footprint (none) -> Connector_PinHeader_2.54mm:PinHeader_1x08_P2.54mm_Vertical
- J5: footprint (none) -> Connector_PinHeader_2.54mm:PinHeader_1x06_P2.54mm_Vertical
- J7: footprint (none) -> Connector_PinHeader_2.54mm:PinHeader_1x10_P2.54mm_Vertical
- J8: footprint (none) -> TerminalBlock:TerminalBlock_MaiXu_MX126-5.0-02P_1x02_P5.00mm
- RV1: footprint (none) -> Potentiometer_THT:Potentiometer_Bourns_3296W_Vertical
Connections:
- net +5V: now also C1.1, C2.1
- net GND: now also C1.2, C2.2
Other:
- note added: "Decoupling Caps"
